File: packages/robocar/unified/hardware/carrier/robocar-unified-carrier/robocar-unified-carrier.kicad_sch (KiCad schematic)
At the start: 38 parts, among them J1 IDC 2x7 head cable, J10 Piezo, J2 IDC 2x7 head cable, J3 XT30 pack in, J4 LM2596 module, J5 Motor left, J6 Motor right, J7 RCWL-1601 front, J8 RCWL-1601 rear, J9 SSD1306 0.91in, U1 XIAO ESP32-S3 Sense, U2 AMS1117-3.3

Commit message: feat(robocar-unified): carrier pre-order changes and three-head panel (#802)
* feat(kicad): circular board cutouts from board.toml [[cutouts]]

robocar-unified's head is sawn off the main board along an L-shaped line
(#750), and a hand saw cannot turn a sharp inside corner: the blade binds and
the corner cracks. A small hole at the corner gives the blade room to turn,
so board.toml needs a way to put a hole through the board. Its copper keepout
band forbids footprints, so the hole is board geometry, not a part.

- board.toml [[cutouts]]: { name, center = [x, y], diameter }, positions
  relative to the outline's top-left corner. boardcheck rejects a missing or
  repeated name, a bad centre or diameter, unknown keys, and a circle that
  is not strictly inside the outline (one touching it would open the edge).
- boardinput passes them through; build_board.py draws each as a circle on
  Edge.Cuts. KiCad's Specctra export then carries the hole as a keepout
  polygon on every signal layer, with the boundary still the outline
  rectangle, so Freerouting routes around it; a test pins both, and fails
  with the drawing removed.

balancebot's board.toml has no cutouts: its DSN export still equals the
fixture.

Co-Authored-By: Claude Opus 5.5 <noreply@anthropic.com>
Claude-Session: https://claude.ai/code/session_01LmLtwHDbHDLXFMLxCn3smf

* feat(parts): reversal-safe head ribbon pinout, UART0 TX carried to a tap

The head ribbon plugs onto unshrouded 2x7 pin headers, so its IDC plug also
fits rotated 180 degrees, which takes pin n to pin 15 - n. With the old
order that put 5 V on XIAO GPIOs. The new order (Lauri, 2026-10-16) pairs
each pin with one that is safe to swap with it:

  (1,14) 5V/5V  (2,13) GND/GND  (3,12) BCLK/LRC  (4,11) STBY/MUX_RST
  (5,10) SCL/SDA  (6,9) UART0 TX/NC  (7,8) DIN/PIEZO

Every non-I2C signal is a XIAO output driving a main-board input, so a
reversed plug only swaps outputs between inputs; I2C swaps with itself, and
TX lands on the unconnected pin 9.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
Parts:
- removed J10: Piezo, Connector_JST:JST_XH_B2B-XH-A_1x02_P2.50mm_Vertical, symbol Device:Buzzer
- added BZ1: Buzzer 12mm, Buzzer_Beeper:Buzzer_12x9.5RM7.6, symbol Device:Buzzer
- added H10, H7, H8, H9: M2, MountingHole:MountingHole_2.2mm_M2_ISO7380, symbol Mechanical:MountingHole
- added J11: Test: 3V3 5V GND VBAT, Connector_PinHeader_2.54mm:PinHeader_1x04_P2.54mm_Vertical, symbol Connector_Generic:Conn_01x04
- added J12: Test: GND SDA SCL RST, Connector_PinHeader_2.54mm:PinHeader_1x04_P2.54mm_Vertical, symbol Connector_Generic:Conn_01x04
- added J13, J14: GND post, Connector_PinHeader_2.54mm:PinHeader_1x02_P2.54mm_Vertical, symbol Connector_Generic:Conn_01x02
- added J15: UART0 TX tap, Connector_PinHeader_2.54mm:PinHeader_1x02_P2.54mm_Vertical, symbol Connector_Generic:Conn_01x02
- added J16, J17: IDC 2x7 head cable, Connector_PinHeader_2.00mm:PinHeader_2x07_P2.00mm_Vertical, symbol Connector_Generic:Conn_02x07_Odd_Even
- added U3, U4: XIAO ESP32-S3 Sense, Seeed_XIAO:XIAO-ESP32-S3-Socket, symbol Seeed_XIAO:XIAO-ESP32-S3-Socket
- C1, C2, C3: LCSC C5162348 -> C96179
- H5, H6: footprint MountingHole:MountingHole_2.2mm_M2 -> MountingHole:MountingHole_2.2mm_M2_ISO7380
- J1, J2: footprint Connector_PinHeader_2.54mm:PinHeader_2x07_P2.54mm_Vertical -> Connector_PinHeader_2.00mm:PinHeader_2x07_P2.00mm_Vertical
Connections:
- net +3V3: now also J11.1 (Pin_1)
- net +5V: now also J1.14 (Pin_14), J11.2 (Pin_2); no longer J1.2 (Pin_2)
- net GND: now also J1.13 (Pin_13), J1.2 (Pin_2), BZ1.2 (-), J11.3 (Pin_3), J12.1 (Pin_1), J13.1 (Pin_1), J13.2 (Pin_2), J14.1 (Pin_1), J14.2 (Pin_2), J15.1 (Pin_1); no longer J1.11 (Pin_11), J1.3 (Pin_3), J1.4 (Pin_4), J1.7 (Pin_7)
- net HEAD_+5V: now also J2.14 (Pin_14); no longer J2.2 (Pin_2)
- net HEAD_GND: now also J2.13 (Pin_13), J2.2 (Pin_2); no longer J2.11 (Pin_11), J2.3 (Pin_3), J2.4 (Pin_4), J2.7 (Pin_7)
- net HEAD_I2C_SCL: now also J2.5 (Pin_5); no longer J2.6 (Pin_6)
- net HEAD_I2C_SDA: now also J2.10 (Pin_10); no longer J2.5 (Pin_5)
- net HEAD_I2S_BCLK: now also J2.3 (Pin_3); no longer J2.8 (Pin_8)
- net HEAD_I2S_DIN: now also J2.7 (Pin_7); no longer J2.10 (Pin_10)
- net HEAD_I2S_LRCLK: now also J2.12 (Pin_12); no longer J2.9 (Pin_9)
- net HEAD_MOTOR_STBY: now also J2.4 (Pin_4); no longer J2.12 (Pin_12)
- net HEAD_MUX_RST: now also J2.11 (Pin_11); no longer J2.14 (Pin_14)
- net HEAD_PIEZO: now also J2.8 (Pin_8); no longer J2.13 (Pin_13)
- net I2C_SCL: now also J1.5 (Pin_5), J12.3 (Pin_3); no longer J1.6 (Pin_6)
- net I2C_SDA: now also J1.10 (Pin_10), J12.2 (Pin_2); no longer J1.5 (Pin_5)
- net I2S_BCLK: now also J1.3 (Pin_3); no longer J1.8 (Pin_8)
- net I2S_DIN: now also J1.7 (Pin_7); no longer J1.10 (Pin_10)
- net I2S_LRCLK: now also J1.12 (Pin_12); no longer J1.9 (Pin_9)
- net MOTOR_STBY: now also J1.4 (Pin_4); no longer J1.12 (Pin_12)
- net MUX_RST: now also J1.11 (Pin_11), J12.4 (Pin_4); no longer J1.14 (Pin_14)
- net PIEZO: now also J1.8 (Pin_8); no longer J1.13 (Pin_13)
- net PIEZO_DRV: now also BZ1.1 (+)
- net VBAT: now also J11.4 (Pin_4)
- net HEAD_UART0_TX: now reaches U1.7 (D6)
- net HEAD_UART0_TX: now also J2.6 (Pin_6)
- new net HEAD2_+5V: J16.1 (Pin_1), J16.14 (Pin_14), U3.14 (VBUS)
- new net HEAD2_GND: J16.13 (Pin_13), J16.2 (Pin_2), U3.13 (GND)
- new net HEAD2_I2C_SCL: J16.5 (Pin_5), U3.6 (D5)
- new net HEAD2_I2C_SDA: J16.10 (Pin_10), U3.5 (D4)
- new net HEAD2_I2S_BCLK: J16.3 (Pin_3), U3.9 (D8)
- new net HEAD2_I2S_DIN: J16.7 (Pin_7), U3.11 (D10)
- new net HEAD2_I2S_LRCLK: J16.12 (Pin_12), U3.10 (D9)
- new net HEAD2_MOTOR_STBY: J16.4 (Pin_4), U3.1 (D0)
- new net HEAD2_MUX_RST: J16.11 (Pin_11), U3.3 (D2)
- new net HEAD2_PIEZO: J16.8 (Pin_8), U3.2 (D1)
- new net HEAD2_UART0_TX: J16.6 (Pin_6), U3.7 (D6)
- new net HEAD3_+5V: J17.1 (Pin_1), J17.14 (Pin_14), U4.14 (VBUS)
- new net HEAD3_GND: J17.13 (Pin_13), J17.2 (Pin_2), U4.13 (GND)
- new net HEAD3_I2C_SCL: J17.5 (Pin_5), U4.6 (D5)
- new net HEAD3_I2C_SDA: J17.10 (Pin_10), U4.5 (D4)
- new net HEAD3_I2S_BCLK: J17.3 (Pin_3), U4.9 (D8)
- new net HEAD3_I2S_DIN: J17.7 (Pin_7), U4.11 (D10)
- new net HEAD3_I2S_LRCLK: J17.12 (Pin_12), U4.10 (D9)
- new net HEAD3_MOTOR_STBY: J17.4 (Pin_4), U4.1 (D0)
- new net HEAD3_MUX_RST: J17.11 (Pin_11), U4.3 (D2)
- new net HEAD3_PIEZO: J17.8 (Pin_8), U4.2 (D1)
- new net HEAD3_UART0_TX: J17.6 (Pin_6), U4.7 (D6)
- new net UART0_TX: J1.6 (Pin_6), J15.2 (Pin_2)
- no-connect marks 16 -> 25
Other:
- moved on the sheet: C1, C2, C3, C4, C5, C7, C8, H1, H2, H3, H4, H5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
