File: packages/robocar/unified/hardware/carrier/robocar-unified-carrier/robocar-unified-carrier.kicad_sch (KiCad schematic)
At the start: 32 parts, among them J1 IDC 2x7 head cable, J10 Piezo, J2 IDC 2x7 head cable, J3 XT30 pack in, J4 LM2596 module, J5 Motor left, J6 Motor right, J7 RCWL-1601 front, J8 RCWL-1601 rear, J9 SSD1306 0.91in, U1 XIAO ESP32-S3 Sense, U2 AMS1117-3.3

Commit message: feat(robocar-unified): combined head and main outline and placement
Replaces #793's row-packed stand-in with a layout: one 100 x 100 mm
rectangle holding the main board and, in the top-right corner, the head
board for the pan-tilt cradle. A 3 mm keepout band under a silkscreen saw
line separates them, so JLCPCB sees a single design and Lauri saws the
head off after delivery.

- Head (30 x 34 mm): the XIAO socket with USB-C at the outer edge, J2
  lying along the bottom edge so the ribbon folds toward the pan axis, and
  two M2 holes for the cradle. It is wider than the planned 24 mm because
  the shrouded 2x7 header is 26.4 mm long.
- Main: M3 holes at its four corners. The TB6612 sits at the left edge,
  with the left motor lead below it and the right motor lead on the right
  edge. J1 is beside the band at the pan-tilt end. Power in, the buck lead,
  the rear rangefinder and the piezo are on the rear edge, and the front
  rangefinder and the OLED lead on the front edge. Each decoupling or bulk
  capacitor is beside the part it serves.
- HEAD_GND gets its own pour region on the head; GND pours the main board.
  The .kicad_dru single-spoke rule now covers both nets.
- Mounting holes are carrier parts, as on balancebot: H1-H4 M3, and H5-H6
  M2 from a new m2-mounting-hole registry entry with its vendored footprint.
- [project] paper is A2, the sheet the schematic writer grows to.

Every dimension is provisional and its board.toml comment says what to
measure. The cradle plate, the chassis plate and the ribbon length are
still unmeasured. The board is routed by Freerouting only so the carrier
gates have a routed board to check; the header still says not to order
it.

Part of #750.

Co-Authored-By: Claude Opus 5.5 <noreply@anthropic.com>
Claude-Session: https://claude.ai/code/session_01LmLtwHDbHDLXFMLxCn3smf
Parts:
- added H1, H2, H3, H4: M3, MountingHole:MountingHole_3.2mm_M3, symbol Mechanical:MountingHole
- added H5, H6: M2, MountingHole:MountingHole_2.2mm_M2, symbol Mechanical:MountingHole
Other:
- moved on the sheet: J1, J10, J2, J3, J4, J5, J6, J7, J8, J9, R1, R2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

Commit message: fix(robocar-unified): fit the head board to the 30 x 30 mm cradle (#797)
* fix(kicad): set a back-side part's silk after flipping it

build_board.py applied [silk] ref_positions before the flip, so the flip
mirrored the label with the footprint: J2's reference landed at y 15.04
instead of the 21.0 board.toml asked for. The flip now comes straight
after Add(), before any silk. A test pins the stored reference offset,
and fails with the old order.

Co-Authored-By: Claude Opus 5.5 <noreply@anthropic.com>
Claude-Session: https://claude.ai/code/session_01LmLtwHDbHDLXFMLxCn3smf

* fix(robocar-unified): fit the head board to the 30 x 30 mm cradle

Lauri measured the cradle's inner height at 30.0 mm as well as its width,
so the head is sawn to 29.5 x 29.5 mm: copper x 72-100, y 0-28, with the
3 mm band and saw lines at x 70.5 and y 29.5.

The XIAO socket and the shrouded IDC header (26.5 mm long) no longer fit
together in 28 mm, with or without the M2 holes. Lauri's choice: J2 and J1
become unshrouded 2x7 pin headers (one registry entry serves both ends),
J2 on the back face beside the XIAO, and the M2 holes go in the two bottom
corners. The ribbon plug is unkeyed on a pin header; the footprint's pin-1
mark carries the orientation on both faces.

HEAD_+5V and HEAD_GND move to the 0.5 mm logic_power class: 1 mm tracks
do not route between the head's pads, and the XIAO and camera draw well
under 1 A. Freerouting also routed head tracks onto the edge, inside
KiCad's 0.5 mm copper-to-edge rule, so 0.5 mm keepouts now line the top,
left and right edges (not the bottom, where J3's courtyard meets it).
The band's move frees the main board's corner, so A2 and C4 return to
their #794 positions.

Board re-placed and re-routed with carrier-board; carrier-check passes
and wrote the stamp. Still provisional: do not order.

Co-Authored-By: Claude Opus 5.5 <noreply@anthropic.com>
Claude-Session: https://claude.ai/code/session_01LmLtwHDbHDLXFMLxCn3smf

* fix(robocar-unified): put the head'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
Parts:
- J1, J2: footprint Connector_IDC:IDC-Header_2x07_P2.54mm_Vertical -> Connector_PinHeader_2.54mm:PinHeader_2x07_P2.54mm_Vertical
Changed lines of the file:
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@@
 			)
 		)
-		(property "Footprint" "Connector_IDC:IDC-Header_2x07_P2.54mm_Vertical"
+		(property "Footprint" "Connector_PinHeader_2.54mm:PinHeader_2x07_P2.54mm_Vertical"
 			(at 266.7 121.92 0)
 			(hide yes)
@@
 			)
 		)
-		(property "Footprint" "Connector_IDC:IDC-Header_2x07_P2.54mm_Vertical"
+		(property "Footprint" "Connector_PinHeader_2.54mm:PinHeader_2x07_P2.54mm_Vertical"
 			(at 320.04 121.92 0)
 			(hide yes)

Commit message: feat(parts): reversal-safe head ribbon pinout, UART0 TX carried to a tap
The head ribbon plugs onto unshrouded 2x7 pin headers, so its IDC plug also
fits rotated 180 degrees, which takes pin n to pin 15 - n. With the old
order that put 5 V on XIAO GPIOs. The new order (Lauri, 2026-10-16) pairs
each pin with one that is safe to swap with it:

  (1,14) 5V/5V  (2,13) GND/GND  (3,12) BCLK/LRC  (4,11) STBY/MUX_RST
  (5,10) SCL/SDA  (6,9) UART0 TX/NC  (7,8) DIN/PIEZO

Every non-I2C signal is a XIAO output driving a main-board input, so a
reversed plug only swaps outputs between inputs; I2C swaps with itself, and
TX lands on the unconnected pin 9. GND drops from four conductors to two;
the head draws well under 1 A. test_registry checks every pair.

Pin 6 now carries D6 (UART0 TX, GPIO43) to J15, a 1x2 GND/TX header on the
main board, where the ROM bootloader's boot log appears at 115200 baud with
no firmware change. In hardware.toml the UART0_TX_PIN [[undrawn]] entry
becomes harness-only and a carrier-only [[nets]] entry wires the role to
J15, so the harness view and WIRING.md are unchanged; D6 leaves the cable's
head_no_connect. D7 (RX) stays open on the head.

netlist.py: a cable entry's no_connect pin (pin 9, "NC") is a spare
conductor, not an MCU pad, and stays open at both ends; before, every cable
pin had to name a XIAO pad.

The board is re-placed and re-routed in a later commit on this branch.

Co-Authored-By: Claude Opus 5.5 <noreply@anthropic.com>
Claude-Session: https://claude.ai/code/session_01LmLtwHDbHDLXFMLxCn3smf
Parts:
- added J15: UART0 TX tap, Connector_PinHeader_2.54mm:PinHeader_1x02_P2.54mm_Vertical, symbol Connector_Generic:Conn_01x02
Connections:
- net +5V: now also J1.14 (Pin_14); no longer J1.2 (Pin_2)
- net GND: now also J1.13 (Pin_13), J1.2 (Pin_2), J15.1 (Pin_1); no longer J1.11 (Pin_11), J1.3 (Pin_3), J1.4 (Pin_4), J1.7 (Pin_7)
- net HEAD_+5V: now also J2.14 (Pin_14); no longer J2.2 (Pin_2)
- net HEAD_GND: now also J2.13 (Pin_13), J2.2 (Pin_2); no longer J2.11 (Pin_11), J2.3 (Pin_3), J2.4 (Pin_4), J2.7 (Pin_7)
- net HEAD_I2C_SCL: now also J2.5 (Pin_5); no longer J2.6 (Pin_6)
- net HEAD_I2C_SDA: now also J2.10 (Pin_10); no longer J2.5 (Pin_5)
- net HEAD_I2S_BCLK: now also J2.3 (Pin_3); no longer J2.8 (Pin_8)
- net HEAD_I2S_DIN: now also J2.7 (Pin_7); no longer J2.10 (Pin_10)
- net HEAD_I2S_LRCLK: now also J2.12 (Pin_12); no longer J2.9 (Pin_9)
- net HEAD_MOTOR_STBY: now also J2.4 (Pin_4); no longer J2.12 (Pin_12)
- net HEAD_MUX_RST: now also J2.11 (Pin_11); no longer J2.14 (Pin_14)
- net HEAD_PIEZO: now also J2.8 (Pin_8); no longer J2.13 (Pin_13)
- net I2C_SCL: now also J1.5 (Pin_5); no longer J1.6 (Pin_6)
- net I2C_SDA: now also J1.10 (Pin_10); no longer J1.5 (Pin_5)
- net I2S_BCLK: now also J1.3 (Pin_3); no longer J1.8 (Pin_8)
- net I2S_DIN: now also J1.7 (Pin_7); no longer J1.10 (Pin_10)
- net I2S_LRCLK: now also J1.12 (Pin_12); no longer J1.9 (Pin_9)
- net MOTOR_STBY: now also J1.4 (Pin_4); no longer J1.12 (Pin_12)
- net MUX_RST: now also J1.11 (Pin_11); no longer J1.14 (Pin_14)
- net PIEZO: now also J1.8 (Pin_8); no longer J1.13 (Pin_13)
- net HEAD_UART0_TX: now reaches U1.7 (D6)
- net HEAD_UART0_TX: now also J2.6 (Pin_6)
- new net UART0_TX: J1.6 (Pin_6), J15.2 (Pin_2)
- no-connect marks 16 -> 17
Other:
- moved on the sheet: R1, R2, R3, R4, R5, R6, R7, R8, R9, U1, U2

Commit message: feat(robocar-unified): test headers, UART0 tap and saw relief hole on the carrier
Lauri's pre-order changes for the carrier (2026-10-16), placed and routed:

- J11, 1x4 supply header: +3V3, +5V, GND, VBAT. VBAT is on an end pin with
  GND as its only neighbour, so a probe slipping off VBAT reaches ground,
  never a logic rail.
- J12, 1x4: GND, I2C SDA, I2C SCL, MUX_RST, on the main board's side of the
  ribbon, upstream of the mux. Each role fans out to its J12 pin as a
  carrier-only [[nets]] entry.
- J13 and J14, 1x2 GND posts for scope ground clips, below the MAX98357A
  and C3, and beside the AMS1117.
- J15, the UART0 TX tap from the previous commit, below J1.
- A 2 mm relief hole ([[cutouts]]) centred on the saw line's inside corner,
  (70.5, 29.5). It lies wholly inside the keepout band, so neither board
  loses copper; it notches the head's empty lower-left corner by 1 mm. The
  two cut lines now stop 0.5 mm short of it, the silkscreen-to-edge
  clearance.

All are through-hole pin headers from the vendored library, hand-soldered,
with no LCSC number; three new registry entries carry their pin orders, and
each pin's net name is on the silkscreen. The supply rails take the new
loads as carrier-only continuations, so the harness view and WIRING.md are
unchanged (just hardware::gen leaves the tree clean).

The brief suggested x 52-66, y 38-50 for J11/J12; that area is under the
PCA9685 module (A2's courtyard), so they sit in a row below it instead. The
first route put J15 there too and Freerouting necked an AIN1 track to
0.15 mm under A2's pads. With J15 moved below J1, clear of the tracks
leaving A2's bottom row, the next route had no necking; no rule changed.
Freerouting does not repeat a route, so that is one run, not proof the
placement prevents it. carrier-check passes: ERC, DRC 0 violations, parity, board check,
stamp written.

Co-Authored-By: Claude Opus 5.5 <noreply@anthropic.com>
Claude-Session: https://claude.ai/code/session_01LmLtwHDbHDLXFMLxCn3smf
Parts:
- added J11: Test: 3V3 5V GND VBAT, Connector_PinHeader_2.54mm:PinHeader_1x04_P2.54mm_Vertical, symbol Connector_Generic:Conn_01x04
- added J12: Test: GND SDA SCL RST, Connector_PinHeader_2.54mm:PinHeader_1x04_P2.54mm_Vertical, symbol Connector_Generic:Conn_01x04
- added J13, J14: GND post, Connector_PinHeader_2.54mm:PinHeader_1x02_P2.54mm_Vertical, symbol Connector_Generic:Conn_01x02
Connections:
- net +3V3: now also J11.1 (Pin_1)
- net +5V: now also J11.2 (Pin_2)
- net GND: now also J11.3 (Pin_3), J12.1 (Pin_1), J13.1 (Pin_1), J13.2 (Pin_2), J14.1 (Pin_1), J14.2 (Pin_2)
- net I2C_SCL: now also J12.3 (Pin_3)
- net I2C_SDA: now also J12.2 (Pin_2)
- net MUX_RST: now also J12.4 (Pin_4)
- net VBAT: now also J11.4 (Pin_4)
Other:
- moved on the sheet: J15, R1, R2, R3, R4, R5, R6, R7, R8, R9, U1, U2

Commit message: feat(robocar-unified): carrier-fab recipe, bulk capacitors JLCPCB can place
`just robocar-unified::carrier-fab` runs carrier-check, then writes the
Gerber zip and the JLCPCB BOM and CPL, as balancebot's recipe does. Its
first run: the Edge.Cuts Gerber has the 2 mm relief circle, both
silkscreens carry both cut lines, J2's outline is on the back silkscreen,
and neither copper Gerber has a coordinate inside the cut band. The fab
output stays git-ignored, as balancebot's does.

Checked every SMD part through JLCPCB's parts search on 2026-10-16:

  C1-C3  C5162348  not in JLCPCB's assembly library; LCSC stock 70
  C7-C8  C8020     22 uF 16 V tantalum, Extended, 46,941 in stock
  U2     C6186     AMS1117-3.3, Basic, 1,129,981
  C4-C5  C49678    100 nF 0805, Basic, 21,360,915
  R2-R9  C17414    10 k 0805, Basic, 56,670,916
  R1     C17408    100 R 0805, Basic, 8,729,662

C1-C3 move to C96179: the same part number (CS1C471M-CRF10, 470 uF 16 V,
8 x 10.5 mm) under another LCSC listing, Extended, 24,687 in stock. The
footprint, value and rating are unchanged. JLCPCB lists no Basic 470 uF or
22 uF 16 V tantalum part, so C1-C3 and C7-C8 stay Extended. The board is
re-placed for the new LCSC field (placement unchanged, re-routed) and
carrier-check passes again: DRC 0 violations.

Co-Authored-By: Claude Opus 5.5 <noreply@anthropic.com>
Claude-Session: https://claude.ai/code/session_01LmLtwHDbHDLXFMLxCn3smf
Parts:
- C1, C2, C3: LCSC C5162348 -> C96179
Changed lines of the file:
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@@
 			)
 		)
-		(property "LCSC" "C5162348"
+		(property "LCSC" "C96179"
 			(at 236.22 35.56 0)
 			(hide yes)
@@
 			)
 		)
-		(property "LCSC" "C5162348"
+		(property "LCSC" "C96179"
 			(at 281.94 35.56 0)
 			(hide yes)
@@
 			)
 		)
-		(property "LCSC" "C5162348"
+		(property "LCSC" "C96179"
 			(at 325.12 35.56 0)
 			(hide yes)

Commit message: feat(robocar-unified): rectangular main board with three head variants (#800)
* feat(kicad): spare head boards on a carrier cable

Lauri wants three head variants on one panel to try in the pan-tilt
cradle. A [[cables]] entry may now list spare_heads, each an mcu_ref and
a head_ref. The netlist gives every spare head its own copy of the MCU
socket and of the head connector, joined by HEAD2_*, HEAD3_* nets with
the same split as HEAD_*: the main board keeps one end, so the spare
heads stay off its nets. head_no_connect and the power-pad-on-a-rail rule
apply to each MCU copy.

The join rejects a malformed spare_heads entry and any spare ref that
repeats another ref. The balancebot netlist is unchanged (its #749
export test still passes byte for byte).

Co-Authored-By: Claude Opus 5.5 <noreply@anthropic.com>
Claude-Session: https://claude.ai/code/session_01LmLtwHDbHDLXFMLxCn3smf

* feat(parts): 2.0 mm head ribbon and a 12 mm board-mount buzzer

The head ribbon moves to a 2.0 mm 2x7 pin header at both ends, mated by a
2.0 mm IDC plug on 1.0 mm-pitch ribbon (Lauri, 2026-10-16). The cradle's
sides carry clips, so the header must sit at the head's top or bottom
edge; at 2.0 mm the 2x7 is 14 x 4 mm and fits across that edge beside the
XIAO, where the 17.8 mm 2.54 mm header does not. The reversal-safe pinout
is unchanged, and the KiCad 2.00 mm footprint numbers odd/even across its
rows like the 2.54 mm one, so a rotated plug still maps pin n to 15 - n.

piezo-buzzer-12mm is Lauri's buzzer: 12 mm, 7.6 mm pin pitch, soldered
to the board. Device:Buzzer names pin 1 "+" and Buzzer_12x9.5RM7.6 prints
"+" beside pad 1, which the registry's polarity tripwire checks.

The vendored subset drops the unused 2.54 mm 2x7 header and adds the two
new footprints.

Co-Authored-By: Claude Opus 5.5 <noreply@anthropic.com>
Claude-Session: https://claude.ai/code/session_01LmLtwHDbHDLXFMLxCn3smf

* docs(rcwl-1601): record the bench-verified pin order

Lauri verified the RCWL-1601 header order, VC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
Parts:
- removed J10: Piezo, Connector_JST:JST_XH_B2B-XH-A_1x02_P2.50mm_Vertical, symbol Device:Buzzer
- added BZ1: Buzzer 12mm, Buzzer_Beeper:Buzzer_12x9.5RM7.6, symbol Device:Buzzer
- added H10, H7, H8, H9: M2, MountingHole:MountingHole_2.2mm_M2_ISO7380, symbol Mechanical:MountingHole
- added J16, J17: IDC 2x7 head cable, Connector_PinHeader_2.00mm:PinHeader_2x07_P2.00mm_Vertical, symbol Connector_Generic:Conn_02x07_Odd_Even
- added U3, U4: XIAO ESP32-S3 Sense, Seeed_XIAO:XIAO-ESP32-S3-Socket, symbol Seeed_XIAO:XIAO-ESP32-S3-Socket
- H5, H6: footprint MountingHole:MountingHole_2.2mm_M2 -> MountingHole:MountingHole_2.2mm_M2_ISO7380
- J1, J2: footprint Connector_PinHeader_2.54mm:PinHeader_2x07_P2.54mm_Vertical -> Connector_PinHeader_2.00mm:PinHeader_2x07_P2.00mm_Vertical
Connections:
- net GND: now also BZ1.2 (-)
- net PIEZO_DRV: now also BZ1.1 (+)
- new net HEAD2_+5V: J16.1 (Pin_1), J16.14 (Pin_14), U3.14 (VBUS)
- new net HEAD2_GND: J16.13 (Pin_13), J16.2 (Pin_2), U3.13 (GND)
- new net HEAD2_I2C_SCL: J16.5 (Pin_5), U3.6 (D5)
- new net HEAD2_I2C_SDA: J16.10 (Pin_10), U3.5 (D4)
- new net HEAD2_I2S_BCLK: J16.3 (Pin_3), U3.9 (D8)
- new net HEAD2_I2S_DIN: J16.7 (Pin_7), U3.11 (D10)
- new net HEAD2_I2S_LRCLK: J16.12 (Pin_12), U3.10 (D9)
- new net HEAD2_MOTOR_STBY: J16.4 (Pin_4), U3.1 (D0)
- new net HEAD2_MUX_RST: J16.11 (Pin_11), U3.3 (D2)
- new net HEAD2_PIEZO: J16.8 (Pin_8), U3.2 (D1)
- new net HEAD2_UART0_TX: J16.6 (Pin_6), U3.7 (D6)
- new net HEAD3_+5V: J17.1 (Pin_1), J17.14 (Pin_14), U4.14 (VBUS)
- new net HEAD3_GND: J17.13 (Pin_13), J17.2 (Pin_2), U4.13 (GND)
- new net HEAD3_I2C_SCL: J17.5 (Pin_5), U4.6 (D5)
- new net HEAD3_I2C_SDA: J17.10 (Pin_10), U4.5 (D4)
- new net HEAD3_I2S_BCLK: J17.3 (Pin_3), U4.9 (D8)
- new net HEAD3_I2S_DIN: J17.7 (Pin_7), U4.11 (D10)
- new net HEAD3_I2S_LRCLK: J17.12 (Pin_12), U4.10 (D9)
- new net HEAD3_MOTOR_STBY: J17.4 (Pin_4), U4.1 (D0)
- new net HEAD3_MUX_RST: J17.11 (Pin_11), U4.3 (D2)
- new net HEAD3_PIEZO: J17.8 (Pin_8), U4.2 (D1)
- new net HEAD3_UART0_TX: J17.6 (Pin_6), U4.7 (D6)
- no-connect marks 17 -> 25
Other:
- moved on the sheet: C1, C2, C3, C4, C5, C7, C8, H1, H2, H3, H4, H5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

Commit message: feat(robocar-unified): MCP23017 socket and GPIO mirror header on the carrier (#803)
* feat(kicad): socket footprints from listed pad positions

A breakout socket's pads come from the pad centres its board page records,
which are read from the vendor's board file. The CJMCU-2317 has no board
file, so its page has no centres to read; its column spacing is a bench
measurement. A [[socket]] table may now give `pad_xy`, each pad's [x, y] in
footprint pad order, in place of `pads`. The outline, courtyard, pad shape
and the inside-the-outline and listed-once checks are unchanged.

The breakout-sockets README also said the courtyard bounds only the pads;
it has covered the module outline since #794.

Co-Authored-By: Claude Opus 5.5 <noreply@anthropic.com>
Claude-Session: https://claude.ai/code/session_01LmLtwHDbHDLXFMLxCn3smf

* docs(boards): record Lauri's OLED pin-order and CJMCU-2317 geometry checks

Lauri checked both fitted modules on 2026-10-16. The 0.91" SSD1306's pin
order (GND, VCC, SCL, SDA) matches the photo read, so its page and the
ssd1306-091-cable entry's source now say so; its other checks stay open.

On the CJMCU-2317 the first-named signal of each double-column row is on
the inner hole, the outer column is one 2.54 mm pitch outside the inner,
and the single column is 15.24 mm from the inner, with 2.54 mm rows. The
page gives those positions, which the carrier socket is built from. The
outline is still an estimate from a photo, and the address, RESET and
pull-up checks stay open. The "no board = key" caveat stays: the layout
model still has no inner row.

Co-Authored-By: Claude Opus 5.5 <noreply@anthropic.com>
Claude-Session: https://claude.ai/code/session_01LmLtwHDbHDLXFMLxCn3smf

* feat(parts): CJMCU-2317 socket and its GPIO mirror header

The robocar carrier takes the MCP23017 module by all 30 holes, so it sits
firmly and every pin reaches copper. CJMCU_2317_Socket lists the hole
positions from Lauri's 2026-10-16 measurement (pad_xy) and the page's
estim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
Parts:
- added A5: CJMCU-2317, Breakout_Sockets:CJMCU_2317_Socket, symbol Connector_Generic:Conn_01x30
- added J18: GPIO A/B, Connector_PinHeader_2.54mm:PinHeader_2x10_P2.54mm_Vertical, symbol Connector_Generic:Conn_02x10_Odd_Even
- added R10, R11: 10k, Resistor_SMD:R_0805_2012Metric_Pad1.20x1.40mm_HandSolder, symbol Device:R
Connections:
- net +3V3: now also A5.11 (Pin_11), A5.24 (Pin_24), A5.30 (Pin_30), J18.2 (Pin_2), R10.1, R11.1
- net GND: now also A5.1 (Pin_1), A5.21 (Pin_21), A5.22 (Pin_22), A5.23 (Pin_23), A5.29 (Pin_29), J18.1 (Pin_1)
- net CH2_SDA: now reaches A3.13 (Pin_13)
- net CH2_SDA: now also A5.27 (Pin_27), R10.2
- net CH2_SCL: now reaches A3.14 (Pin_14)
- net CH2_SCL: now also A5.28 (Pin_28), R11.2
- new net EXP_GPA0: A5.3 (Pin_3), J18.5 (Pin_5)
- new net EXP_GPA1: A5.4 (Pin_4), J18.7 (Pin_7)
- new net EXP_GPA2: A5.5 (Pin_5), J18.9 (Pin_9)
- new net EXP_GPA3: A5.6 (Pin_6), J18.11 (Pin_11)
- new net EXP_GPA4: A5.7 (Pin_7), J18.13 (Pin_13)
- new net EXP_GPA5: A5.8 (Pin_8), J18.15 (Pin_15)
- new net EXP_GPA6: A5.9 (Pin_9), J18.17 (Pin_17)
- new net EXP_GPA7: A5.10 (Pin_10), J18.19 (Pin_19)
- new net EXP_GPB0: A5.13 (Pin_13), J18.6 (Pin_6)
- new net EXP_GPB1: A5.14 (Pin_14), J18.8 (Pin_8)
- new net EXP_GPB2: A5.15 (Pin_15), J18.10 (Pin_10)
- new net EXP_GPB3: A5.16 (Pin_16), J18.12 (Pin_12)
- new net EXP_GPB4: A5.17 (Pin_17), J18.14 (Pin_14)
- new net EXP_GPB5: A5.18 (Pin_18), J18.16 (Pin_16)
- new net EXP_GPB6: A5.19 (Pin_19), J18.18 (Pin_18)
- new net EXP_GPB7: A5.20 (Pin_20), J18.20 (Pin_20)
- new net EXP_INTA: A5.2 (Pin_2), J18.3 (Pin_3)
- new net EXP_INTB: A5.12 (Pin_12), J18.4 (Pin_4)
Other:
- moved on the sheet: BZ1, C1, C2, C3, C4, C5, C7, C8, H1, H10, H2, H3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

Commit message: feat(robocar-unified): backport the integrated carrier's pre-fab review fixes (#812)
Works through #810's ten findings on the socketed carrier:

- [fanout] with required vias on the bulk capacitors, C4, C5 and the
  AMS1117 and its capacitors: GND vias go from 1 to 11, and no SMD
  ground pad is left without one
- F1, a 3 A hold, 16 V 1812 PTC (C883162) between the XT30 and VBAT;
  the harness keeps its unfused VBAT rail
- mux channel pull-ups R2-R11 from 10 kOhm to 2.2 kOhm (C17520, Basic)
  for the 300 ns Fast-mode rise time; the harness docs follow
- head 2's top saw band reaches 1 mm past its cut; head 3's stays at
  0.5 mm, because a wider band left HEAD3_PIEZO unroutable past J17
- silkscreen at 1.0 mm where DRC allows it
- README records each finding's outcome, including the not-applicable
  ones (cutoff, LED brightness, decoupling distance); WIRING.md gains
  the low-battery and 5 V current-budget notes from SNVS124G

Board re-placed and re-routed; every carrier gate passes and the stamp
is rewritten.


Claude-Session: https://claude.ai/code/session_01HMYrZm6JVcVgRypdr4Jojz

Co-authored-by: Claude <noreply@anthropic.com>
Parts:
- added F1: 3A hold 16V, Fuse:Fuse_1812_4532Metric_Pad1.30x3.40mm_HandSolder, symbol Device:Polyfuse
- R10, R11, R2, R3, R4, R5, R6, R7, R8, R9: value 10k -> 2.2k; LCSC C17414 -> C17520
Connections:
- net VBAT: now also F1.2; no longer J3.2 (Pin_2)
- new net PACK_IN: F1.1, J3.2 (Pin_2)
Other:
- moved on the sheet: H1, H10, H2, H3, H4, H5, H6, H7, H8, H9, J1, J11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
