File: packages/robocar/unified/hardware/carrier/robocar-unified-carrier/robocar-unified-carrier.kicad_sch (KiCad schematic)
At the start: 56 parts, among them J1 IDC 2x7 head cable, J11 Test: 3V3 5V GND VBAT, J12 Test: GND SDA SCL RST, J13 GND post, J14 GND post, J15 UART0 TX tap, J16 IDC 2x7 head cable, J17 IDC 2x7 head cable, J18 GPIO A/B, J2 IDC 2x7 head cable, J3 XT30 pack in, J4 LM2596 module, J5 Motor left, J6 Motor right, J7 RCWL-1601 front, J8 RCWL-1601 rear, J9 SSD1306 0.91in, U1 XIAO ESP32-S3 Sense, U2 AMS1117-3.3, U3 XIAO ESP32-S3 Sense, U4 XIAO ESP32-S3 Sense

Commit message: fix(robocar-unified): pre-order fixes to the carrier PCB (#823)
* feat(kicad): [fanout] own pads take a via of their own

A pad joined by a fixed track to another pad that has a via counted as
having one, so the integrated carrier's buck GND pin (U10:1), tied under
the package to C11, never got a via beside it. An `own` pad ignores that
chain and takes its own via (TI's first layout rule for the TPS563208).

Co-Authored-By: Claude Opus 5.5 <noreply@anthropic.com>
Claude-Session: https://claude.ai/code/session_01DgeoMcrSCUfJwedu77q6oo

* fix(robocar-unified-integrated): fix the power paths the layout review found

The pre-fab layout review of the integrated carrier found the buck's output
capacitors 75 mm of track from L1 and the pack input on a 0.25 mm track,
neither visible to a gate. Fixed tracks in board.toml now:

- chain C13, C14 and C20 onto L1's output pad, and run the trunk and a 1 mm
  east branch (C7, the LDO, FB1) from that node;
- give the feedback divider its own sense track from C20;
- carry PACK_IN on 2 mm from the XT30 to F1;
- run C12 straight into L1 so U10's GND pin gets its own via.

C5, C6 and C18 move beside the pins they decouple, C21 adds 10 uF at the
TB6612FNG's VM1, the GND pour stops 1 mm short of the mouse-bite slot, and
R26 becomes 36 k so EN is guaranteed on by 6.3 V rather than 7.2 V. The
README records each finding with before and after measurements, and that
the pack takes an external 2S BMS.

Routed with KiCad 10.0.7 (the stamp records it), not the pinned 10.0.6.

Co-Authored-By: Claude Opus 5.5 <noreply@anthropic.com>
Claude-Session: https://claude.ai/code/session_01DgeoMcrSCUfJwedu77q6oo

* docs(robocar-unified-integrated): correct the layout fixes table

The M1 row said VM1 and the servos reach L1 with no via. They still share
one 0.8/0.4 mm via: the measuring script joined B.Cu track ends to F.Cu
tracks they only cross. The m1, m2 and m5 rows take the second review's
layer-aware measurements, and its findings are listed as still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
Parts:
- added C6: 100nF, Capacitor_SMD:C_0805_2012Metric_Pad1.18x1.45mm_HandSolder, symbol Device:C
- added D1: B5819W, Diode_SMD:D_SOD-123, symbol Device:D_Schottky
- added R12, R13: 2.2k, Resistor_SMD:R_0805_2012Metric_Pad1.20x1.40mm_HandSolder, symbol Device:R
- F1: value 3A hold 16V -> 4A hold 16V; LCSC C883162 -> C47263807
- J4: footprint Connector_JST:JST_XH_B4B-XH-A_1x04_P2.50mm_Vertical -> Connector_JST:JST_VH_B4P-VH_1x04_P3.96mm_Vertical
Connections:
- net +3V3: now also C6.1, R12.1, R13.1
- net +5V: now also D1.2 (A); no longer J1.1 (Pin_1), J1.14 (Pin_14)
- net GND: now also C6.2
- net I2C_SCL: now also R13.2
- net I2C_SDA: now also R12.2
- net HEAD2_+5V renamed HEAD2_XIAO_5V
- net HEAD3_+5V renamed HEAD3_XIAO_5V
- net HEAD_+5V renamed HEAD_XIAO_5V
- new net XIAO_5V: D1.1 (K), J1.1 (Pin_1), J1.14 (Pin_14)
Other:
- moved on the sheet: C7, C8, F1, H1, H10, H2, H3, H4, H5, H6, H7, H8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
