File: packages/robocar/unified-integrated/hardware/carrier/robocar-unified-integrated-carrier/robocar-unified-integrated-carrier.kicad_sch (KiCad schematic)
At the start: 77 parts, among them J1 IDC 2x7 head cable, J11 Test: 3V3 5V GND VBAT, J12 Test: GND SDA SCL RST, J13 GND post, J14 GND post, J15 UART0 TX tap, J18 GPIO A/B, J19 Speaker, J2 IDC 2x7 head cable, J20 Pan servo (SG90), J21 Tilt servo (SG90), J22 Left RGB LED, J23 Right RGB LED, J3 XT30 pack in, J5 Motor left, J6 Motor right, J7 RCWL-1601 front, J8 RCWL-1601 rear, J9 SSD1306 0.91in, U1 XIAO ESP32-S3 Sense, U10 TPS563201, U2 AMS1117-3.3, U5 TCA9548APWR, U6 PCA9685PW, U7 TB6612FNG, U8 MAX98357AETE+, U9 MCP23017-E/SS

Commit message: feat(robocar-unified): lay out and route the integrated carrier board
The integrated carrier now has a board: a 64.5 x 76 mm main board (the
socketed carrier's is about 70.5 x 100 mm) and the 29.5 mm head square
on one panel, placed in board.toml, routed by Freerouting and poured.
It passes every carrier gate with KiCad 10.0.6: ERC, DRC with schematic
parity, netlist parity, the board check and the stamp.

The MAX98357A takes 5V through a ferrite bead (FB1) as its own net,
AMP_5V: Freerouting gives each net one width, and the amplifier's
0.5 mm-pitch pins would otherwise cap the whole 5V rail at 0.25 mm. Net
classes follow the narrowest pins on each net; the .kicad_pro allows
0.15 mm tracks, where Freerouting necks down at fine-pitch pads.

check-added-large-files now skips .kicad_pcb: a routed, poured board
is about 1 MB.

Co-Authored-By: Claude Opus 5.5 <noreply@anthropic.com>
Claude-Session: https://claude.ai/code/session_01AoNL8UeiSeWCVt1Bs1JLVr
Parts:
- added FB1: 600R@100MHz 2A, Inductor_SMD:L_0805_2012Metric_Pad1.05x1.20mm_HandSolder, symbol Device:FerriteBead
Connections:
- net +5V: now also FB1.1; no longer C17.1, C18.1, C3.1, U8.4 (~{SD_MODE}), U8.7 (VDD), U8.8 (VDD)
- new net AMP_5V: C17.1, C18.1, C3.1, FB1.2, U8.4 (~{SD_MODE}), U8.7 (VDD), U8.8 (VDD)
Other:
- moved on the sheet: H1, H2, H3, H4, H5, H6, J1, J11, J12, J13, J14, J15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

Commit message: feat(robocar-unified-integrated): 5V trunk and pour, SMD bulk capacitors
- 1.5 mm 5V trunk from L1 to C2 beside the TB6612FNG's VM pins, inside a
  +5V pour on F.Cu above GND; B.Cu stays the GND plane.
- Buck GND as a fixed track from U10's GND pin, under the package, to
  input capacitor C11; C9-C11 turned so their GND pads face it.
- C1-C3 470 uF electrolytics become 22 uF MnO2 tantalums (3528): TI caps
  the TPS563201's low-ESR output capacitance at 68 uF, and their ESR
  keeps them out of the D-CAP2 loop and damps FB1. Low-ESR polymer was
  rejected for the same reason.
- C19 100 uF electrolytic on VBAT for hot-plug damping.
- R12 54.9k per SLVSD90B Table 7-2 (4.98 V).
- Floorplan: PCA9685 and its headers swapped with the motor driver block.

Main-board courtyards: 2234 mm^2 (-58 % against the socketed carrier).

Co-Authored-By: Claude Opus 5.5 <noreply@anthropic.com>
Claude-Session: https://claude.ai/code/session_01AoNL8UeiSeWCVt1Bs1JLVr
Parts:
- added C19: 100uF 25V, Capacitor_SMD:CP_Elec_6.3x7.7, symbol Device:C_Polarized
- C1, C2, C3: value 470uF 16V -> 22uF 16V; footprint Capacitor_SMD:CP_Elec_8x10.5 -> Capacitor_Tantalum_SMD:CP_EIA-3528-21_Kemet-B_HandSolder; LCSC C96179 -> C8020
- R12: value 56.2k -> 54.9k
Connections:
- net GND: now also C19.2
- net VBAT: now also C19.1
Other:
- moved on the sheet: FB1, H1, H2, H3, H4, H5, H6, J1, J11, J12, J13, J14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

Commit message: feat(robocar-unified-integrated): add the two spare head boards
The socketed carrier's three head boards, in the same column moved 6 mm
left: head 1 (U1/J2, header on the back), head 2 (U3/J16, front) and
head 3 (U4/J17, back at the top), with M2 holes H5-H10 and each head's
own ground pour (HEAD_GND, HEAD2_GND, HEAD3_GND). The outline grows to
94 x 100 mm; the main board stays 64.5 x 76 and the strip below it is
waste behind a keepout and a cut line.

Co-Authored-By: Claude Opus 5.5 <noreply@anthropic.com>
Claude-Session: https://claude.ai/code/session_01AoNL8UeiSeWCVt1Bs1JLVr
Parts:
- added H10, H7, H8, H9: M2, MountingHole:MountingHole_2.2mm_M2_ISO7380, symbol Mechanical:MountingHole
- added J16, J17: IDC 2x7 head cable, Connector_PinHeader_2.00mm:PinHeader_2x07_P2.00mm_Vertical, symbol Connector_Generic:Conn_02x07_Odd_Even
- added U3, U4: XIAO ESP32-S3 Sense, Seeed_XIAO:XIAO-ESP32-S3-Socket, symbol Seeed_XIAO:XIAO-ESP32-S3-Socket
Connections:
- new net HEAD2_+5V: J16.1 (Pin_1), J16.14 (Pin_14), U3.14 (VBUS)
- new net HEAD2_GND: J16.13 (Pin_13), J16.2 (Pin_2), U3.13 (GND)
- new net HEAD2_I2C_SCL: J16.5 (Pin_5), U3.6 (D5)
- new net HEAD2_I2C_SDA: J16.10 (Pin_10), U3.5 (D4)
- new net HEAD2_I2S_BCLK: J16.3 (Pin_3), U3.9 (D8)
- new net HEAD2_I2S_DIN: J16.7 (Pin_7), U3.11 (D10)
- new net HEAD2_I2S_LRCLK: J16.12 (Pin_12), U3.10 (D9)
- new net HEAD2_MOTOR_STBY: J16.4 (Pin_4), U3.1 (D0)
- new net HEAD2_MUX_RST: J16.11 (Pin_11), U3.3 (D2)
- new net HEAD2_PIEZO: J16.8 (Pin_8), U3.2 (D1)
- new net HEAD2_UART0_TX: J16.6 (Pin_6), U3.7 (D6)
- new net HEAD3_+5V: J17.1 (Pin_1), J17.14 (Pin_14), U4.14 (VBUS)
- new net HEAD3_GND: J17.13 (Pin_13), J17.2 (Pin_2), U4.13 (GND)
- new net HEAD3_I2C_SCL: J17.5 (Pin_5), U4.6 (D5)
- new net HEAD3_I2C_SDA: J17.10 (Pin_10), U4.5 (D4)
- new net HEAD3_I2S_BCLK: J17.3 (Pin_3), U4.9 (D8)
- new net HEAD3_I2S_DIN: J17.7 (Pin_7), U4.11 (D10)
- new net HEAD3_I2S_LRCLK: J17.12 (Pin_12), U4.10 (D9)
- new net HEAD3_MOTOR_STBY: J17.4 (Pin_4), U4.1 (D0)
- new net HEAD3_MUX_RST: J17.11 (Pin_11), U4.3 (D2)
- new net HEAD3_PIEZO: J17.8 (Pin_8), U4.2 (D1)
- new net HEAD3_UART0_TX: J17.6 (Pin_6), U4.7 (D6)
- no-connect marks 19 -> 27
Other:
- moved on the sheet: J1, J11, J12, J13, J14, J15, J18, J19, J2, J20, J21, J22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

Commit message: fix(robocar-unified-integrated): address the pre-fab review
Layout (review B1): the +5V F.Cu pour cut F.Cu GND into islands around
every chip in the power half, and the board had one GND via, so their
ground pads reached the B.Cu plane through 0.19-0.25 mm tracks. The pour
is gone; [fanout] adds 48 GND vias, required on every power-path pad;
the MAX98357A's GND pins and GAIN_SLOT tie to its exposed pad, which
takes an in-pad via. Pours stop 1 mm short of every cut line.

Power stage:
- TPS563208 (forced-continuous: sinks motor regeneration) for the
  TPS563201; same pins and Table 7-2 values.
- L1 4.7 uH +/-20 % (the 3.3 uH part's +/-30 % can fall below 3.3 uH);
  a third 22 uF output capacitor, C20.
- EN divider R25/R26 (100k/30k): on near 6.2 V, off near 4.9 V.
- F1 3 A PTC between the XT30 and VBAT.

Placement: the EN and feedback dividers beside their pins above U10,
C13/C14/C20 east of L1, FB1 beside the amplifier, C8 beside the LDO,
C7 and C14 away from the y 76 cut. RGB green/blue series 47 ohm.
Silkscreen text 1.0 mm (0.8 mm where it cannot fit), stroke >= 0.16 mm.
Freerouting's neck-downs below the 0.15 mm minimum are widened after
routing. README: the review's open items, the 6.7 V dropout and the 5 V
current budget.

Co-Authored-By: Claude Opus 5.5 <noreply@anthropic.com>
Claude-Session: https://claude.ai/code/session_01AoNL8UeiSeWCVt1Bs1JLVr
Parts:
- added C20: 22uF 16V, Capacitor_SMD:C_0805_2012Metric_Pad1.18x1.45mm_HandSolder, symbol Device:C
- added F1: 3A hold 16V, Fuse:Fuse_1812_4532Metric_Pad1.30x3.40mm_HandSolder, symbol Device:Polyfuse
- added R25: 100k, Resistor_SMD:R_0805_2012Metric_Pad1.20x1.40mm_HandSolder, symbol Device:R
- added R26: 30k, Resistor_SMD:R_0805_2012Metric_Pad1.20x1.40mm_HandSolder, symbol Device:R
- L1: value 3.3uH -> 4.7uH
- R18, R19, R21, R22: value 220 -> 47
- U10: value TPS563201 -> TPS563208
Connections:
- net +5V: now also C20.1
- net GND: now also C20.2, R26.2
- net VBAT: now also F1.2, R25.1; no longer J3.2 (Pin_2), U10.5 (EN)
- new net BUCK_EN: R25.2, R26.1, U10.5 (EN)
- new net PACK_IN: F1.1, J3.2 (Pin_2)
Other:
- moved on the sheet: C12, C13, C14, C15, C16, C17, C18, C19, FB1, H1, H10, H2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

Commit message: feat(robocar-unified-integrated): LCSC parts for every SMD line, fiducials, 2.2k I2C pull-ups
Every SMD part now has an LCSC number (Basic where one exists), so
carrier-fab's bom-jlc.csv and cpl-jlc.csv cover all 56 placements. Three
fiducials on the main board. The I2C pull-ups follow the socketed
carrier's 2.2 kOhm (#810). Board re-placed, re-routed and checked with
KiCad 10.0.6; README records the part table, rotations and a cost estimate.

Refs #808

Co-Authored-By: Claude Opus 5.5 <noreply@anthropic.com>
Claude-Session: https://claude.ai/code/session_01NQBHdVJbY6M136w1wzwDHy
Parts:
- added FID1, FID2, FID3: Fiducial, Fiducial:Fiducial_1mm_Mask2mm, symbol Mechanical:Fiducial
- C10, C16, C17, C9: LCSC (none) -> C15850
- C13, C14, C20: value 22uF 16V -> 22uF 25V; LCSC (none) -> C45783
- C19: value 100uF 25V -> 100uF 35V; LCSC (none) -> C2836437
- F1: LCSC (none) -> C883162
- FB1: value 600R@100MHz 2A -> 220R@100MHz 2A; LCSC (none) -> C85840
- L1: LCSC (none) -> C2044594
- R10, R11, R14, R15, R2, R3, R4, R5, R6, R7, R8, R9: value 10k -> 2.2k; LCSC C17414 -> C17520
- R12: LCSC (none) -> C17747
- R17, R20, R23, R24: LCSC (none) -> C17557
- R18, R19, R21, R22: LCSC (none) -> C17714
- R25: LCSC (none) -> C149504
- R26: LCSC (none) -> C17621
- U10: LCSC (none) -> C468250
- U5: LCSC (none) -> C130026
- U6: LCSC (none) -> C2678753
- U7: LCSC (none) -> C88224
- U8: LCSC (none) -> C910544
- U9: LCSC (none) -> C506653
Other:
- moved on the sheet: H1, H10, H2, H3, H4, H5, H6, H7, H8, H9, J1, J11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

Commit message: fix(robocar-unified-integrated): fix the power paths the layout review found (#818)
* feat(kicad): [fanout] own pads take a via of their own

A pad joined by a fixed track to another pad that has a via counted as
having one, so the integrated carrier's buck GND pin (U10:1), tied under
the package to C11, never got a via beside it. An `own` pad ignores that
chain and takes its own via (TI's first layout rule for the TPS563208).

Co-Authored-By: Claude Opus 5.5 <noreply@anthropic.com>
Claude-Session: https://claude.ai/code/session_01DgeoMcrSCUfJwedu77q6oo

* fix(robocar-unified-integrated): fix the power paths the layout review found

The pre-fab layout review of the integrated carrier found the buck's output
capacitors 75 mm of track from L1 and the pack input on a 0.25 mm track,
neither visible to a gate. Fixed tracks in board.toml now:

- chain C13, C14 and C20 onto L1's output pad, and run the trunk and a 1 mm
  east branch (C7, the LDO, FB1) from that node;
- give the feedback divider its own sense track from C20;
- carry PACK_IN on 2 mm from the XT30 to F1;
- run C12 straight into L1 so U10's GND pin gets its own via.

C5, C6 and C18 move beside the pins they decouple, C21 adds 10 uF at the
TB6612FNG's VM1, the GND pour stops 1 mm short of the mouse-bite slot, and
R26 becomes 36 k so EN is guaranteed on by 6.3 V rather than 7.2 V. The
README records each finding with before and after measurements, and that
the pack takes an external 2S BMS.

Routed with KiCad 10.0.7 (the stamp records it), not the pinned 10.0.6.

Co-Authored-By: Claude Opus 5.5 <noreply@anthropic.com>
Claude-Session: https://claude.ai/code/session_01DgeoMcrSCUfJwedu77q6oo

* docs(robocar-unified-integrated): correct the layout fixes table

The M1 row said VM1 and the servos reach L1 with no via. They still share
one 0.8/0.4 mm via: the measuring script joined B.Cu track ends to F.Cu
tracks they only cross. The m1, m2 and m5 rows take the second review's
layer-aware measurements, and its findings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
Parts:
- added C21: 10uF 25V, Capacitor_SMD:C_0805_2012Metric_Pad1.18x1.45mm_HandSolder, symbol Device:C
- R26: value 30k -> 36k; LCSC C17621 -> C4360
Connections:
- net +5V: now also C21.1
- net GND: now also C21.2
Other:
- moved on the sheet: F1, FB1, FID1, FID2, FID3, H1, H10, H2, H3, H4, H5, H6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

Commit message: fix(robocar-unified-integrated): fix the second layout review's findings
- VBAT into the buck on 1.0/0.5 mm vias only; the sense track and the FB1
  branch move east and C10 0.3 mm east to make room, and B.Cu route keepouts
  hold VBAT off the feedback divider and a stray GND run off its via.
- +5V takes its own net class with 1.0/0.5 mm vias.
- C15 turned so its GND pad faces U7's GND pin (20.6 mm to 5.4 mm), and its
  GND pad now needs a fanout via.
- Head pours start 1 mm short of the mouse-bite slot: 0.70 mm to every hole.
- R12 54.9 k to 56 k: 5.07 V, at or above the TB6612FNG's VM >= 5 V row.
- C11 and C10 swap, so the 10 uF sits beside VIN.

The README's before/after table is re-measured with layer-aware scripts.

Co-Authored-By: Claude Opus 5.5 <noreply@anthropic.com>
Claude-Session: https://claude.ai/code/session_01DgeoMcrSCUfJwedu77q6oo
Parts:
- C10: value 10uF 25V -> 100nF; LCSC C15850 -> C49678
- C11: value 100nF -> 10uF 25V; LCSC C49678 -> C15850
- R12: value 54.9k -> 56k; LCSC C17747 -> C17756
Changed lines of the file:
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@@
 			)
 		)
-		(property "Value" "10uF 25V"
+		(property "Value" "100nF"
 			(at 495.808 41.91 0)
 			(show_name no)
@@
 			)
 		)
-		(property "LCSC" "C15850"
+		(property "LCSC" "C49678"
 			(at 497.84 35.56 0)
 			(hide yes)
@@
 			)
 		)
-		(property "Value" "100nF"
+		(property "Value" "10uF 25V"
 			(at 541.528 41.91 0)
 			(show_name no)
@@
 			)
 		)
-		(property "LCSC" "C49678"
+		(property "LCSC" "C15850"
 			(at 543.56 35.56 0)
 			(hide yes)
@@
 			)
 		)
-		(property "Value" "54.9k"
+		(property "Value" "56k"
 			(at 131.064 173.99 0)
 			(show_name no)
@@
 			)
 		)
-		(property "LCSC" "C17747"
+		(property "LCSC" "C17756"
 			(at 132.08 167.64 0)
 			(hide yes)

Commit message: fix(robocar-unified-integrated): put a B5819W between 5V and the XIAO's 5V pad
The socketed carrier's pre-fab review found the ribbon's 5V tied straight to
the XIAO's 5V pad, which is its USB-C VBUS; this carrier shares the cable and
the fault. With a USB cable on the head, the PC's port and the buck fed each
other. D1, as the balancebot carrier's, feeds a new XIAO_5V net on J1:1 and
J1:14; the head nets follow it (HEAD*_XIAO_5V). Routed and checked: every
gate passes, and the README table is re-measured on this route.

Co-Authored-By: Claude Opus 5.5 <noreply@anthropic.com>
Claude-Session: https://claude.ai/code/session_01DgeoMcrSCUfJwedu77q6oo
Parts:
- added D1: B5819W, Diode_SMD:D_SOD-123, symbol Device:D_Schottky
Connections:
- net +5V: now also D1.2 (A); no longer J1.1 (Pin_1), J1.14 (Pin_14)
- net HEAD2_+5V renamed HEAD2_XIAO_5V
- net HEAD3_+5V renamed HEAD3_XIAO_5V
- net HEAD_+5V renamed HEAD_XIAO_5V
- new net XIAO_5V: D1.1 (K), J1.1 (Pin_1), J1.14 (Pin_14)
Other:
- moved on the sheet: F1, FB1, FID1, FID2, FID3, H1, H10, H2, H3, H4, H5, H6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
