File: packages/robocar/unified-integrated/hardware/carrier/robocar-unified-integrated-carrier/robocar-unified-integrated-carrier.kicad_sch (KiCad schematic)
At the start: 96 parts, among them J1 IDC 2x7 head cable, J11 Test: 3V3 5V GND VBAT, J12 Test: GND SDA SCL RST, J13 GND post, J14 GND post, J15 UART0 TX tap, J16 IDC 2x7 head cable, J17 IDC 2x7 head cable, J18 GPIO A/B, J19 Speaker, J2 IDC 2x7 head cable, J20 Pan servo (SG90), J21 Tilt servo (SG90), J22 Left RGB LED, J23 Right RGB LED, J3 XT30 pack in, J5 Motor left, J6 Motor right, J7 RCWL-1601 front, J8 RCWL-1601 rear, J9 SSD1306 0.91in, U1 XIAO ESP32-S3 Sense, U10 TPS563208, U2 AMS1117-3.3, U3 XIAO ESP32-S3 Sense, U4 XIAO ESP32-S3 Sense, U5 TCA9548APWR, U6 PCA9685PW, U7 TB6612FNG, U8 MAX98357AETE+, U9 MCP23017-E/SS

Commit message: fix(robocar-unified-integrated): fix the third layout review's findings
- N9: Q1, a DMP3013SFV P-MOSFET, between the XT30 and F1 for reverse-
  polarity protection, gate to GND through R27 (10k), on fixed tracks:
  PACK_IN 1.2 mm through the slot between F1 and the XT30's GND pin, the
  source pads tied and 1.5 mm into F1.
- S3: U8's GND pin 3 takes a fanout via of its own, so the exposed pad's
  via is no longer the amplifier ground's only way to the plane
  (`carrier-measure cuts GND J3:1`: none). A tie from pin 11 to C17 boxed
  in SPK_VO- on every route and was dropped.
- S1: rebuilt with pcb/silk.py: thinnest silkscreen line 0.150 mm.
- S4b: B.Cu under the 5V trunk kept GND by router keepouts, with one gap
  where VBAT crosses under it.
- N7: router keepouts keep tracks out from under head 3's screw heads;
  the nearest copper to H9 and H10 is now HEAD3_GND pour at 0.25 mm.
- A B.Cu keepout under U8's exposed-pad via, which Freerouting cannot see.
- [pour] stitch at 5 mm: the 141.7 mm2 top-left piece at J7:4 joins the
  main plane. Two top-left pieces and the servo-ground piece (N1) are
  still joined only by tracks; see the README.

Routed by Freerouting 2.5.0 with 0 unrouted, checked with KiCad 10.0.7
(the stamp records it), not the pinned 10.0.6; origin/main's stamp was
also written by 10.0.7.

Co-Authored-By: Claude Opus 5.5 <noreply@anthropic.com>
Claude-Session: https://claude.ai/code/session_013Jm7qdC6rgErFatzdYrBYY
Parts:
- added Q1: DMP3013SFV, Package_SON:Diodes_PowerDI3333-8, symbol Transistor_FET:DMP3013SFV
- added R27: 10k, Resistor_SMD:R_0805_2012Metric_Pad1.20x1.40mm_HandSolder, symbol Device:R
Connections:
- net GND: now also R27.2
- net PACK_IN: now also Q1.5 (D); no longer F1.1
- new net PACK_RP: F1.1, Q1.1 (S), Q1.2 (S), Q1.3 (S)
- new net PFET_GATE: Q1.4 (G), R27.1
Other:
- moved on the sheet: R1, R10, R11, R12, R13, R14, R15, R16, R17, R18, R19, R2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
