File: packages/robocar/unified-integrated/hardware/carrier/robocar-unified-integrated-carrier/robocar-unified-integrated-carrier.kicad_pcb (KiCad board)
At the start: 2 copper layers, 94 x 100 mm, 109 parts, among them J1 IDC 2x7 head cable, J11 Test: 3V3 5V GND VBAT, J12 Test: GND SDA SCL RST, J13 GND post, J14 GND post, J15 UART0 TX tap, J16 IDC 2x7 head cable, J17 IDC 2x7 head cable, J18 GPIO A/B, J19 Speaker, J2 IDC 2x7 head cable, J20 Pan servo (SG90), J21 Tilt servo (SG90), J22 Left RGB LED, J23 Right RGB LED, J3 XT30 pack in, J5 Motor left, J6 Motor right, J7 RCWL-1601 front, J8 RCWL-1601 rear, J9 SSD1306 0.91in, U1 XIAO ESP32-S3 Sense, U10 TPS563208, U2 AMS1117-3.3, U3 XIAO ESP32-S3 Sense, U4 XIAO ESP32-S3 Sense, U5 TCA9548APWR, U6 PCA9685PW, U7 TB6612FNG, U8 MAX98357AETE+, U9 MCP23017-E/SS

Commit message: fix(robocar-unified-integrated): put a B5819W between 5V and the XIAO's 5V pad
The socketed carrier's pre-fab review found the ribbon's 5V tied straight to
the XIAO's 5V pad, which is its USB-C VBUS; this carrier shares the cable and
the fault. With a USB cable on the head, the PC's port and the buck fed each
other. D1, as the balancebot carrier's, feeds a new XIAO_5V net on J1:1 and
J1:14; the head nets follow it (HEAD*_XIAO_5V). Routed and checked: every
gate passes, and the README table is re-measured on this route.

Co-Authored-By: Claude Opus 5.5 <noreply@anthropic.com>
Claude-Session: https://claude.ai/code/session_01DgeoMcrSCUfJwedu77q6oo
Parts:
- added D1: B5819W, Diode_SMD:D_SOD-123, F.Cu at (146.0, 110.0)
Connections:
- net HEAD2_+5V renamed HEAD2_XIAO_5V
- net HEAD3_+5V renamed HEAD3_XIAO_5V
- net HEAD_+5V renamed HEAD_XIAO_5V
- J1 pad 1: +5V -> XIAO_5V
- J1 pad 14: +5V -> XIAO_5V
Routing:
- net XIAO_5V: track 0.00 -> 29.4 mm, vias 0 -> 1
- net I2C_SDA: track 62.6 -> 42.8 mm, vias 2 -> 1
- net EXP_INTA: track 13.1 -> 29.2 mm, vias 0 -> 1
- net EXP_GPA6: track 19.4 -> 33.6 mm, vias 1 -> 3
- net MOTOR_STBY: track 74.1 -> 87.7 mm, vias 3 -> 1
- net I2C_SCL: track 39.3 -> 51.0 mm, vias 4 -> 3
- net PIEZO: track 49.5 -> 60.1 mm
- net I2S_BCLK: track 45.8 -> 55.6 mm, vias 0 -> 1
- net EXP_INTB: track 30.4 -> 22.6 mm, vias 1 -> 0
- net EXP_GPA7: track 31.7 -> 24.2 mm, vias 3 -> 2
- net EXP_GPA5: track 25.0 -> 17.7 mm
- net GND: track 435.4 -> 442.5 mm, vias 47 -> 52
- net HEAD_I2S_DIN: track 23.8 -> 30.3 mm
- net EXP_GPB0: track 17.2 -> 23.2 mm
- net EXP_GPB2: track 31.9 -> 26.3 mm
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
Commit message: fix(robocar-unified-integrated): fix the third layout review's findings
- N9: Q1, a DMP3013SFV P-MOSFET, between the XT30 and F1 for reverse-
  polarity protection, gate to GND through R27 (10k), on fixed tracks:
  PACK_IN 1.2 mm through the slot between F1 and the XT30's GND pin, the
  source pads tied and 1.5 mm into F1.
- S3: U8's GND pin 3 takes a fanout via of its own, so the exposed pad's
  via is no longer the amplifier ground's only way to the plane
  (`carrier-measure cuts GND J3:1`: none). A tie from pin 11 to C17 boxed
  in SPK_VO- on every route and was dropped.
- S1: rebuilt with pcb/silk.py: thinnest silkscreen line 0.150 mm.
- S4b: B.Cu under the 5V trunk kept GND by router keepouts, with one gap
  where VBAT crosses under it.
- N7: router keepouts keep tracks out from under head 3's screw heads;
  the nearest copper to H9 and H10 is now HEAD3_GND pour at 0.25 mm.
- A B.Cu keepout under U8's exposed-pad via, which Freerouting cannot see.
- [pour] stitch at 5 mm: the 141.7 mm2 top-left piece at J7:4 joins the
  main plane. Two top-left pieces and the servo-ground piece (N1) are
  still joined only by tracks; see the README.

Routed by Freerouting 2.5.0 with 0 unrouted, checked with KiCad 10.0.7
(the stamp records it), not the pinned 10.0.6; origin/main's stamp was
also written by 10.0.7.

Co-Authored-By: Claude Opus 5.5 <noreply@anthropic.com>
Claude-Session: https://claude.ai/code/session_013Jm7qdC6rgErFatzdYrBYY
Parts:
- added Q1: DMP3013SFV, Package_SON:Diodes_PowerDI3333-8, F.Cu at (113.0, 157.5)
- added R27: 10k, Resistor_SMD:R_0805_2012Metric_Pad1.20x1.40mm_HandSolder, F.Cu at (109.6, 157.0)
Connections:
- F1 pad 1: PACK_IN -> PACK_RP
Routing:
- net HEAD3_MOTOR_STBY: track 41.3 -> 21.3 mm, vias 1 -> 0
- net HEAD3_PIEZO: track 36.7 -> 19.0 mm, vias 1 -> 0
- net +3V3: track 264.0 -> 247.8 mm, vias 2 -> 3
- net EXP_GPA7: track 24.2 -> 40.0 mm
- net I2C_SCL: track 51.0 -> 38.1 mm
- net EXP_GPA6: track 33.6 -> 21.2 mm, vias 3 -> 2
- net EXP_INTA: track 29.2 -> 17.0 mm
- net MOTOR_STBY: track 87.7 -> 75.9 mm, vias 1 -> 2
- net I2C_SDA: track 42.8 -> 53.7 mm
- net HEAD3_XIAO_5V: track 28.4 -> 38.5 mm, vias 2 -> 1
- net I2S_LRCLK: track 57.8 -> 65.3 mm, vias 1 -> 2
- net EXP_GPA0: track 20.7 -> 13.2 mm
- net HEAD3_UART0_TX: track 37.3 -> 44.5 mm
- net MUX_RST: track 63.3 -> 70.4 mm
- net EXP_GPA5: track 17.7 -> 24.3 mm
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
Commit message: fix(robocar-unified-integrated): hand-saw panel, servo ground tie, VBAT width
The seventh pre-fab layout review's findings, and Lauri's choice of saw
mode:

- [panel] mode = "saw": one outline, which JLCPCB counts as one design.
  Head 3's band stays at y 71.0 (71.5 leaves HEAD3_PIEZO unrouted with the
  keepouts under H9 and H10).
- SF2: a fixed 0.8 mm F.Cu track from U6's GND pin 1 to the servo header
  J21:3, through a gap R17 opens by moving 0.6 mm north. J20:3 to J3:1
  ~12.50 -> ~2.64 mOhm (`carrier-measure resistance`). The track starts on
  U6:1 so that pin leaves Freerouting's netlist: ending there, its keepout
  boxed the pin in and GND lost 15 connections. A second tie from J20:3 to
  J21:3 walled F.Cu across the board and +3V3 lost 24; dropped.
- SF1: the router keepout beside VBAT's input via stops at y 68.65; at 68.8
  it necked the 10.3 mm B.Cu run under L1 to 0.6 mm. That run is 0.8 mm
  now; VBAT F1:2 to U10:3 ~26.4 -> ~24.2 mOhm, 0.6 mm still narrowest, on
  F.Cu beside the input via.
- J11:3 is back on the main plane (~11.06 -> ~3.48 mOhm to J3:1).

The head cable's +5V path got worse (to D1 ~52.5 -> ~67.5 mOhm, 3 vias):
signals crossing the new ground tie take B.Cu. Four more routes of the same
board.toml gave the same paths; the README says so.

Freerouting 2.5.0: 0 unrouted. Checked with KiCad 10.0.7 (the stamp records
it), not the pinned 10.0.6.

Co-Authored-By: Claude Opus 5.5 <noreply@anthropic.com>
Claude-Session: https://claude.ai/code/session_013Jm7qdC6rgErFatzdYrBYY
Parts:
- removed MB1, MB10, MB11, MB12, MB13, MB14, MB2, MB3, MB4, MB5, MB6, MB7, MB8, MB9: MouseBites, MouseBites
- moved R17 0.60 mm to (113.4, 126.9)
Routing:
- net GND: track 436.4 -> 486.1 mm, vias 77 -> 90
- net EXP_GPA7: track 40.0 -> 20.9 mm
- net MUX_RST: track 70.4 -> 52.2 mm, vias 2 -> 4
- net EXP_GPB4: track 19.6 -> 37.1 mm, vias 2 -> 1
- net HEAD2_XIAO_5V: track 48.6 -> 66.1 mm
- net HEAD2_MUX_RST: track 39.2 -> 23.7 mm
- net SERVO_TILT: track 34.9 -> 22.7 mm, vias 0 -> 1
- net EXP_GPB1: track 17.2 -> 28.8 mm
- net I2C_SCL: track 38.1 -> 49.3 mm, vias 3 -> 1
- net HEAD_XIAO_5V: track 53.5 -> 43.0 mm
- net MOTOR_STBY: track 75.9 -> 67.9 mm
- net PIEZO: track 61.6 -> 53.7 mm, vias 1 -> 2
- net XIAO_5V: track 24.0 -> 30.8 mm
- net I2S_DIN: track 54.9 -> 48.2 mm, vias 1 -> 0
- net EXP_GPB0: track 17.7 -> 23.5 mm, vias 0 -> 1
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Other:
- outline, holes or cut-outs redrawn
- board text added: "CUT"
