File: packages/robocar/unified-integrated/hardware/carrier/robocar-unified-integrated-carrier/robocar-unified-integrated-carrier.kicad_pcb (KiCad board)
At the start: 2 copper layers, 94 x 100 mm, 110 parts, among them J1 IDC 2x7 head cable, J11 Test: 3V3 5V GND VBAT, J12 Test: GND SDA SCL RST, J13 GND post, J14 GND post, J15 UART0 TX tap, J16 IDC 2x7 head cable, J17 IDC 2x7 head cable, J18 GPIO A/B, J19 Speaker, J2 IDC 2x7 head cable, J20 Pan servo (SG90), J21 Tilt servo (SG90), J22 Left RGB LED, J23 Right RGB LED, J3 XT30 pack in, J5 Motor left, J6 Motor right, J7 RCWL-1601 front, J8 RCWL-1601 rear, J9 SSD1306 0.91in, U1 XIAO ESP32-S3 Sense, U10 TPS563208, U2 AMS1117-3.3, U3 XIAO ESP32-S3 Sense, U4 XIAO ESP32-S3 Sense, U5 TCA9548APWR, U6 PCA9685PW, U7 TB6612FNG, U8 MAX98357AETE+, U9 MCP23017-E/SS

Commit message: fix(robocar-unified-integrated): fix the sixth and seventh pre-fab reviews' findings (#832)
* feat(kicad): derive a JLCPCB rotation from chosen pads

KiCad's PowerDI3333-8 draws the drain pad and its fingers as one pad 5,
centred on the drain; LCSC numbers the fingers 5-8, so its pad 5 is a
corner finger and lcsc_rotation found no turn within 0.5 mm (best 1.14 mm).
`--pads 1,2,3,4` matches only the listed KiCad pads; the rotation table
entry records `pads`, and `--check` re-derives on the same pads.

Co-Authored-By: Claude Opus 5.5 <noreply@anthropic.com>
Claude-Session: https://claude.ai/code/session_013Jm7qdC6rgErFatzdYrBYY

* fix(kicad): cap a fanout stub at its pad's narrow side

A fanout stub starts at the pad's centre, so its round end cap is as wide
as the stub. From the MAX98357A's 0.25 mm pins at 0.5 mm pitch, a 0.4 mm
stub came 0.175 mm from the next pin on every ray, under the 0.2 mm
clearance, and no GND pin of the amplifier could take a via of its own.
`fanout.stub_width` keeps the stub no wider than the pad.

Co-Authored-By: Claude Opus 5.5 <noreply@anthropic.com>
Claude-Session: https://claude.ai/code/session_013Jm7qdC6rgErFatzdYrBYY

* feat(kicad): add the DMP3013SFV P-MOSFET to the parts registry

A 30 V P-channel MOSFET in PowerDI3333-8 for a pack's reverse-polarity
switch where the SOT-223 ZXMP4A16G runs too hot: 17 mohm max at VGS -4.5 V
(Diodes DS40141 Rev. 5-2), VGSS +-25 V. LCSC C264098 (Extended).

The symbol and footprint are vendored at KiCad 10.0.6. The installed KiCad
is 10.0.7, which `kicad.vendor --update` refuses, so the subset was rebuilt
through `vendor.update()` with the two footprints that differ in 10.0.7
(Fiducial_1mm_Mask2mm, the MAX98357A's TQFN-16) taken from the committed
10.0.6 copies: the diff only adds files. The DMP3013SFV symbol block is
byte-identical to kicad-symbols 10.0.6's Transistor_FET.kicad_symdir, and
the footprint to kicad-footprints 10.0.6's.

Its JLCPCB rotation (270) is matched on pins 1-4 (`--pads`): LCSC n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
Parts:
- removed MB1, MB10, MB11, MB12, MB13, MB14, MB2, MB3, MB4, MB5, MB6, MB7, MB8, MB9: MouseBites, MouseBites
- added Q1: DMP3013SFV, Package_SON:Diodes_PowerDI3333-8, F.Cu at (113.0, 157.5)
- added R27: 10k, Resistor_SMD:R_0805_2012Metric_Pad1.20x1.40mm_HandSolder, F.Cu at (109.6, 157.0)
- moved R17 0.60 mm to (113.4, 126.9)
Connections:
- F1 pad 1: PACK_IN -> PACK_RP
Routing:
- net GND: track 442.5 -> 486.1 mm, vias 52 -> 90
- net HEAD3_MOTOR_STBY: track 41.3 -> 21.3 mm, vias 1 -> 0
- net MOTOR_STBY: track 87.7 -> 67.9 mm, vias 1 -> 2
- net +3V3: track 264.0 -> 246.2 mm, vias 2 -> 3
- net EXP_GPB4: track 19.4 -> 37.1 mm
- net HEAD3_PIEZO: track 36.7 -> 19.0 mm, vias 1 -> 0
- net HEAD2_XIAO_5V: track 48.6 -> 66.1 mm
- net HEAD2_MUX_RST: track 39.2 -> 23.7 mm
- net EXP_INTA: track 29.2 -> 17.0 mm, vias 1 -> 0
- net I2C_SDA: track 42.8 -> 54.5 mm, vias 1 -> 3
- net EXP_GPB1: track 17.1 -> 28.8 mm
- net SERVO_TILT: track 34.2 -> 22.7 mm
- net MUX_RST: track 63.3 -> 52.2 mm, vias 2 -> 4
- net EXP_GPA6: track 33.6 -> 23.0 mm, vias 3 -> 1
- net HEAD_XIAO_5V: track 53.2 -> 43.0 mm
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Other:
- outline, holes or cut-outs redrawn
- board text added: "CUT"
