File: packages/robotics/balancebot/hardware/carrier/balancebot-carrier/balancebot-carrier.kicad_pcb (KiCad board)
At the start: 2 copper layers, 90 x 62 mm, 19 parts, among them J1 JST-XH pack in, J2 LM2596 module, J3 GY-521 MPU6050, J4 Motor left, J5 Motor right, U1 XIAO RP2350

Commit message: fix(balancebot): pre-order fixes to the carrier PCB
From the adversarial pre-order review:

- S1: VMOT, EN and DIR printed at the ends of each DRV8825 socket, since a
  Pololu-format module fits turned 180 degrees; README check "VMOT text =
  module's VMOT pin".
- S2: footprint silkscreen at 0.15 mm (was 0.10-0.127 mm), from the
  build_board.py floor; board-level "+" by C1 and C2 and "K" by D1.
- S3: J2 labelled IN+, -, 5V, - and J4/J5 A1, A2, B1, B2 by their pads;
  README: meter the buck lead before the first plug-in.
- S4: reverse-polarity and short protection at J1, as Lauri chose: F1 (3 A
  hold PTC, BSMD1812-300-24V) and Q1 (ZXMP4A16G P-MOSFET, drain to F1,
  source to VBAT, gate to GND through R4). Datasheet answers in the
  hardware.toml comment and the README. J1 turns 180 degrees so its BAT+
  pad faces F1; "+"/"-" move below it.
- N2: VBAT is fixed F.Cu tracks, 1.5 mm, with no via (was one 1.0/0.5 mm
  via in series to A2, C2 and R2 after 94 mm, and 30 mm of B.Cu).
- N4: C3 at the ADC pin, 2.3 mm from U1:1 (was 24.5 mm).
- N5: [fanout] vias at the SMD ground pads and [pour] stitch vias on a 5 mm
  grid: 118 GND vias (was 3).
- N6: a .kicad_dru rule keeps the pour 3.5 mm from each M3 hole's centre
  (was 1.85 mm, 0.25 mm from the hole).
- N1: README minimums measured on the routed board.
- N9: README notes the DRV8825's 8.2 V minimum and a ~9 V firmware cutoff
  (#747).

The perfboard layout gains F1, Q1 and R4 and a "Pack input" step.

Co-Authored-By: Claude Opus 5.5 <noreply@anthropic.com>
Claude-Session: https://claude.ai/code/session_01DgeoMcrSCUfJwedu77q6oo
Parts:
- added F1: 3A hold 24V, Fuse:Fuse_1812_4532Metric_Pad1.30x3.40mm_HandSolder, F.Cu at (129.5, 155.5)
- added Q1: ZXMP4A16G, Package_TO_SOT_SMD:SOT-223-3_TabPin2, F.Cu at (138.0, 155.5)
- added R4: 10k, Resistor_SMD:R_0805_2012Metric_Pad1.20x1.40mm_HandSolder, F.Cu at (145.0, 158.5)
- moved C3 28.7 mm to (134.0, 106.4), turned to 180 degrees
- moved J1 2.50 mm to (122.5, 155.5), turned to 180 degrees
Connections:
- J1 pad 1: VBAT -> PACK_IN
Routing:
- net VBAT: track 144.4 -> 204.2 mm, vias 1 -> 0
- net GND: track 226.9 -> 262.9 mm, vias 3 -> 120
- net PACK_FUSED: track 0.00 -> 9.43 mm
- net IMU_SCL: track 37.3 -> 29.7 mm
- net DIR_R: track 34.2 -> 41.1 mm
- net PACK_IN: track 0.00 -> 4.78 mm
- net PACK_SENSE: track 36.4 -> 32.3 mm
- net PFET_GATE: track 0.00 -> 3.14 mm
- net IMU_SDA: track 34.5 -> 33.1 mm
- net XIAO_5V: track 53.1 -> 51.7 mm
- net NENABLE: track 49.2 -> 48.2 mm, vias 0 -> 1
Other:
- board text added: "5V"
- board text added: "A1"
- board text added: "A2"
- board text added: "B1"
- board text added: "B2"
- board text added: "DIR"
- board text added: "EN"
- board text added: "IN+"
- board text added: "K"
- board text added: "VMOT"
