File: packages/robotics/balancebot/hardware/carrier/balancebot-carrier/balancebot-carrier.kicad_pcb (KiCad board)
At the start: 2 copper layers, 90 x 62 mm, 19 parts, among them J1 XT30 pack in, J2 LM2596 module, J3 GY-521 MPU6050, J4 Motor left, J5 Motor right, U1 XIAO RP2350

Commit message: feat(balancebot): SMD passives on the carrier, with JLCPCB assembly files (#753)
R1-R3 and C3 move to 0805 hand-solder pads, D1 to a B5819W in SOD-123 and
C1/C2 to 100 uF 35 V 6.3x7.7 mm SMD electrolytics. Each symbol carries an
LCSC number (all JLC Basic except C1/C2), so the same board can be
hand-soldered or assembled by JLCPCB; carrier-fab now also writes a
JLC-format BOM and CPL holding only those seven parts. Modules, sockets and
connectors stay through-hole.

build_board.py copies custom symbol fields onto the footprints (hidden, on
F.Fab) so DRC schematic parity holds. The board was regenerated and
rerouted; ERC, DRC (0 violations, 0 unconnected, 0 parity) and the
pin_config.h cross-check pass.


Claude-Session: https://claude.ai/code/session_01UKeVTQabun2jCo4T7rwoBH

Co-authored-by: Claude Opus 5.5 <noreply@anthropic.com>
Parts:
- C1, C2: value 100uF 25V -> 100uF 35V; footprint Capacitor_THT:CP_Radial_D8.0mm_P3.50mm -> Capacitor_SMD:CP_Elec_6.3x7.7
- C3: footprint Capacitor_THT:C_Disc_D5.0mm_W2.5mm_P5.00mm -> Capacitor_SMD:C_0805_2012Metric_Pad1.18x1.45mm_HandSolder
- D1: value 1N5819 -> B5819W; footprint Diode_THT:D_DO-41_SOD81_P10.16mm_Horizontal -> Diode_SMD:D_SOD-123
- R1, R2, R3: footprint Resistor_THT:R_Axial_DIN0207_L6.3mm_D2.5mm_P10.16mm_Horizontal -> Resistor_SMD:R_0805_2012Metric_Pad1.20x1.40mm_HandSolder
- moved D1 5.00 mm to (171.0, 150.0)
- moved R1 5.00 mm to (131.5, 131.0)
- moved R2 5.00 mm to (162.0, 104.0)
- moved R3 5.00 mm to (162.0, 109.0)
- moved C3 2.50 mm to (161.5, 114.5)
- moved C1 1.75 mm to (109.8, 144.0)
- moved C2 1.75 mm to (177.8, 114.0)
Routing:
- net GND: track 201.7 -> 210.7 mm, vias 0 -> 2
- net +3V3: track 82.6 -> 77.7 mm
- net VBAT: track 135.9 -> 131.9 mm, vias 0 -> 1
- net PACK_SENSE: track 39.6 -> 35.7 mm
- net XIAO_5V: track 51.3 -> 55.0 mm, vias 0 -> 1
- net BUCK_5V: track 13.6 -> 10.1 mm, vias 0 -> 1
- net NENABLE: track 49.0 -> 48.5 mm, vias 0 -> 2

Commit message: fix(balancebot): seat the GY-521 right side up and take the pack on JST-XH (#770)
* fix(balancebot): seat the GY-521 right side up and take the pack on JST-XH

J3 sat at the front edge of the GY-521's outline, so the module hung
rearward from it. Component side up, that put VCC on the wrong end of
the socket; component side down, Z pointed down and the firmware's
atan2(accel_x, accel_z) would read about 180 deg upright. Moving J3 to
the rear edge (y 33 -> 47) puts VCC on pin 1 with the module component
side up, its X arrow toward FWD and Z up, as WIRING.md and the firmware
expect.

The XT30 is replaced by a JST-XH 2-pin (no XT30 plugs on hand). The new
registry entry names its pins BAT+/BAT- rather than +/-: the JST-XH
footprint prints no polarity for the tripwire to prove, so the carrier
silkscreen prints + and - over the pads instead. The XT30 entry and its
vendored footprint stay for the registry tests.

The DRV8825 and GY-521 pin orders in the pre-order checks are confirmed
against the HW-216 carriers and the GY-521 on hand (#748).

Co-Authored-By: Claude Opus 5.5 <noreply@anthropic.com>
Claude-Session: https://claude.ai/code/session_01V4exdSPypzhBpgNeQYJDD5

* docs(parts): record the GY-521 and DRV8825 pin orders as checked

Both were read off the fitted modules on 2026-10-14 (#748); the
registry's source lines still said "from memory" and "not yet checked".
The test_bad_values mutation now anchors on the source key rather than
its old wording.

Co-Authored-By: Claude Opus 5.5 <noreply@anthropic.com>
Claude-Session: https://claude.ai/code/session_01V4exdSPypzhBpgNeQYJDD5

* fix(balancebot): point the perfboard GY-521's X arrow forward

The perfboard socket sat on row 1 with pin 1 at its right end, so the
module, component side up, hung rearward and its X arrow pointed to the
rear, against the README and the firmware's X-forward mounting. The
socket now runs I7-P7 with VCC at I7 and the module extends toward
row 1, matching the carrier's J3.

Co-Authored-By: Cla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
Parts:
- J1: value XT30 pack in -> JST-XH pack in; footprint Connector_AMASS:AMASS_XT30PW-M_1x02_P2.50mm_Horizontal -> Connector_JST:JST_XH_B2B-XH-A_1x02_P2.50mm_Vertical
- moved J3 14.0 mm to (136.1, 147.0)
- moved J1 7.67 mm to (120.0, 155.5), turned to 0 degrees
Connections:
- J1 pad 1: GND -> VBAT
- J1 pad 2: VBAT -> GND
Routing:
- net IMU_SCL: track 16.5 -> 37.3 mm
- net GND: track 210.7 -> 226.9 mm, vias 2 -> 3
- net IMU_SDA: track 19.1 -> 34.5 mm
- net +3V3: track 77.7 -> 92.2 mm
- net IMU_INT: track 25.8 -> 39.8 mm
- net VBAT: track 131.9 -> 144.4 mm
- net DIR_R: track 37.0 -> 34.2 mm, vias 0 -> 1
- net XIAO_5V: track 55.0 -> 53.1 mm
- net NENABLE: track 48.5 -> 49.2 mm, vias 2 -> 0
- net PACK_SENSE: track 35.7 -> 36.4 mm
Other:
- board text added: "+"
- board text added: "-"

Commit message: fix(balancebot): pre-order carrier fixes, reverse-polarity input, stitching vias (#822)
* feat(kicad): [fanout] own pads take a via of their own

A pad joined by a fixed track to another pad that has a via counted as
having one, so the integrated carrier's buck GND pin (U10:1), tied under
the package to C11, never got a via beside it. An `own` pad ignores that
chain and takes its own via (TI's first layout rule for the TPS563208).

Co-Authored-By: Claude Opus 5.5 <noreply@anthropic.com>
Claude-Session: https://claude.ai/code/session_01DgeoMcrSCUfJwedu77q6oo

* fix(robocar-unified-integrated): fix the power paths the layout review found

The pre-fab layout review of the integrated carrier found the buck's output
capacitors 75 mm of track from L1 and the pack input on a 0.25 mm track,
neither visible to a gate. Fixed tracks in board.toml now:

- chain C13, C14 and C20 onto L1's output pad, and run the trunk and a 1 mm
  east branch (C7, the LDO, FB1) from that node;
- give the feedback divider its own sense track from C20;
- carry PACK_IN on 2 mm from the XT30 to F1;
- run C12 straight into L1 so U10's GND pin gets its own via.

C5, C6 and C18 move beside the pins they decouple, C21 adds 10 uF at the
TB6612FNG's VM1, the GND pour stops 1 mm short of the mouse-bite slot, and
R26 becomes 36 k so EN is guaranteed on by 6.3 V rather than 7.2 V. The
README records each finding with before and after measurements, and that
the pack takes an external 2S BMS.

Routed with KiCad 10.0.7 (the stamp records it), not the pinned 10.0.6.

Co-Authored-By: Claude Opus 5.5 <noreply@anthropic.com>
Claude-Session: https://claude.ai/code/session_01DgeoMcrSCUfJwedu77q6oo

* docs(robocar-unified-integrated): correct the layout fixes table

The M1 row said VM1 and the servos reach L1 with no via. They still share
one 0.8/0.4 mm via: the measuring script joined B.Cu track ends to F.Cu
tracks they only cross. The m1, m2 and m5 rows take the second review's
layer-aware measurements, and its find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
Parts:
- added D2: BZT52C15, Diode_SMD:D_SOD-123, F.Cu at (144.0, 155.5)
- added F1: 3A hold 24V, Fuse:Fuse_1812_4532Metric_Pad1.30x3.40mm_HandSolder, F.Cu at (129.5, 155.5)
- added Q1: ZXMP4A16G, Package_TO_SOT_SMD:SOT-223-3_TabPin2, F.Cu at (138.0, 155.5)
- added R4: 10k, Resistor_SMD:R_0805_2012Metric_Pad1.20x1.40mm_HandSolder, F.Cu at (145.0, 159.0)
- moved C3 28.7 mm to (134.0, 106.4), turned to 180 degrees
- moved J1 2.50 mm to (122.5, 155.5), turned to 180 degrees
Connections:
- J1 pad 1: VBAT -> PACK_IN
Routing:
- net VBAT: track 144.4 -> 207.1 mm, vias 1 -> 0
- net GND: track 226.9 -> 264.0 mm, vias 3 -> 120
- net PACK_FUSED: track 0.00 -> 9.43 mm
- net IMU_SCL: track 37.3 -> 29.7 mm
- net DIR_R: track 34.2 -> 41.1 mm
- net PFET_GATE: track 0.00 -> 6.27 mm
- net PACK_IN: track 0.00 -> 4.78 mm
- net PACK_SENSE: track 36.4 -> 32.3 mm
- net IMU_SDA: track 34.5 -> 33.1 mm
- net XIAO_5V: track 53.1 -> 51.7 mm
- net NENABLE: track 49.2 -> 48.2 mm, vias 0 -> 1
Other:
- board text added: "5V"
- board text added: "A1"
- board text added: "A2"
- board text added: "B1"
- board text added: "B2"
- board text added: "DIR"
- board text added: "EN"
- board text added: "IN+"
- board text added: "K"
- board text added: "VMOT"
